Commit message: 根据line进行抓取导航

File: src/robot_urdf/urdf/robot.urdf (robot description, URDF)
Before this commit: robot robot, 5 links, 4 joints
Links:
- link base_link: geometry visual box size=0.40 0.40 0.150
- link left_front_link: geometry visual cylinder length=0.07 radius=0.05
- link left_wheel_link: geometry visual cylinder length=0.07 radius=0.05
- link right_front_link: geometry visual cylinder length=0.07 radius=0.05
- link right_wheel_link: geometry visual cylinder length=0.07 radius=0.05
